Commit message: 十字追加

File: monitor_catch/urdf/robot_arm.urdf (robot description, URDF)
Before this commit: robot robot_arm, 7 links, 6 joints
Links:
- link hand_link: geometry visual box size=0.1 0.2 0.1
- link lower_module_link: geometry visual box size=1.39 0.2 0.028
- link middle_module_link: geometry visual box size=0.02 1.1 0.1575
- link platform_link: geometry visual box size=0.134 0.2 0.201
Joints:
- joint base_lower_joint: origin xyz=0.1 -0.695 0.014 rpy=0 0 0 -> xyz=0.606 0 -0.014 rpy=0 0 0
- joint lower_platform: axis 0 1 0 -> 1 0 0
- joint middle_end: axis 1 0 0 -> 0 1 0; limit lower=-0.606 upper=0.606 effort=2.00 velocity=2.00 -> lower=-0.414425 upper=0.414425 effort=2.00 velocity=2.00
- joint platform_middle: axis 1 0 0 -> 0 1 0; limit lower=-0.606 upper=0.606 effort=2.00 velocity=2.00 -> lower=-0.414425 upper=0.414425 effort=2.00 velocity=2.00

Commit message: 諸々進捗

File: monitor_catch/urdf/robot_arm.urdf (robot description, URDF)
Before this commit: robot robot_arm, 7 links, 6 joints
Links:
- link end_effector_link: geometry visual box size=0.4 0.1 0.12
- link hand_link: geometry visual box size=0.1 0.15 0.1
Joints:
- joint end_wrest: origin xyz=0 0.25 0 rpy=0 0 0 -> xyz=0.25 0 0 rpy=0 0 0
- joint middle_end: origin xyz=0 0.21 0 rpy=0 0 0 -> xyz=0.21 0 0 rpy=0 0 0
- joint wrest_hand: origin xyz=0 0.1 -0.15 rpy=0 0 0 -> xyz=0.1 0 -0.15 rpy=0 0 0
